Commit message: successful simulation of 'modularized' erlecopter model for future spawning of multiple drones

File: ardupilot_sitl_gazebo_plugin/urdf/erlecopter.xacro (robot description, xacro)
@@ -1,6 +1,8 @@
 <?xml version="1.0"?>
 <robot name="erlecopter" xmlns:xacro="http://ros.org/wiki/xacro">
+	<arg name="nspace" default=""/>
   <!-- Properties -->
-  <xacro:property name="namespace" value="erlecopter" />
+  <xacro:property name="namespace" value="$(arg nspace)/erlecopter" />
+  <xacro:property name="bot_name" value="erlecopter" />
   <xacro:property name="rotor_velocity_slowdown_sim" value="10" />
   <xacro:property name="mesh_file" value="erlecopter.dae" />
@@ -155,5 +157,5 @@
   <xacro:include filename="$(find ardupilot_sitl_gazebo_plugin)/urdf/sensors/lidar_sensor.urdf.xacro" />
    <xacro:lidar_sensor
-    name="sonar2"
+    name="lidar"
     parent="base_link"
     ros_topic="sonar_front"

File: ardupilot_sitl_gazebo_plugin/urdf/erlecopter_base.xacro (robot description, xacro)
@@ -1,85 +1,83 @@
 <?xml version="1.0"?>
 <robot name="erlecopter" xmlns:xacro="http://ros.org/wiki/xacro">
-  <xacro:include filename="$(find rotors_description)/urdf/component_snippets.xacro" />
-  <!-- Instantiate erlecopter "mechanics" -->
-  <xacro:include filename="$(find ardupilot_sitl_gazebo_plugin)/urdf/erlecopter.xacro" />
-  <!-- Specify reference parameters for GNSS receiver. -->
-  <xacro:include filename="$(find ardupilot_sitl_gazebo_plugin)/urdf/gps_home_location.xacro" />
-  <!-- Reference heading is equivalent to rotating Gazebo's map.
-       We do not use it for we would loose the match X=North, Y=West -->
-  <!-- in degrees, 0 so North is towards positive X values, and East is towards negative Y values -->
-  <xacro:property name="referenceHeading" value="0" />
-  <!-- Instantiate a controller. -->
-  <xacro:controller_plugin_macro
-    namespace="${namespace}"
-    imu_sub_topic="imu"
-    >
-  </xacro:controller_plugin_macro>
-  <!-- Mount an ADIS16448 IMU. -->
-  <xacro:imu_plugin_macro
-    namespace="${namespace}"
-    imu_suffix=""
-    parent_link="base_link"
-    imu_topic="imu"
-    mass_imu_sensor="0.015"
-    gyroscope_noise_density="0.0003394"
-    gyroscopoe_random_walk="0.000038785"
-    gyroscope_bias_correlation_time="1000.0"
-    gyroscope_turn_on_bias_sigma="0.0087"
-    accelerometer_noise_density="0.004"
-    accelerometer_random_walk="0.006"
-    accelerometer_bias_correlation_time="300.0"
-    accelerometer_turn_on_bias_sigma="0.1960"
-  >
-    <inertia ixx="0.00001" ixy="0.0" ixz="0.0" iyy="0.00001" iyz="0.0" izz="0.00001" />
-    <origin xyz="0 0 0" rpy="0 0 0" />
-  </xacro:imu_plugin_macro>
-  <!-- Mount a GNSS receiver. -->
-  <gazebo>
-    <plugin name="${namespace}_gps_sim" filename="libhector_gazebo_ros_gps.so">
-      <alwaysOn>true</alwaysOn>
-      <topicName>${namespace}/fix</topicName>
-      <velocityTopicName>${namespace}/fix_velocity</velocityTopicName>
-      <referenceLatitude>${referenceLatitude}</referenceLatitude>
-      <referenceLongitude>${referenceLongitude}</referenceLongitude>
-      <referenceHeading>${referenceHeading}</referenceHeading>
-      <referenceAltitude>${referenceAltitude}</referenceAltitude>
-      <!-- Sensor errors model for GPS Position measures -->
-      <!-- Units: [m], and [1/s] for drift frequency -->
-      <!-- For now, use Ardupilot's internal error models -->
-      <offset>0 0 0</offset>
-      <drift>0 0 0</drift>
-      <driftFrequency>0 0 0</driftFrequency>
-      <gaussianNoise>0 0 0</gaussianNoise>
-      <scaleError>1 1 1</scaleError>
-      <!-- Note:
-       For the moment there is no barometer, so axis Z of the GPS is
-       used as a barometer sensor (with the according error model) -->
-      <!-- Sensor errors model for GPS Velocity measures -->
-      <!-- Units: [m/s], and [1/s] for drift frequency -->
-      <!-- For now, use Ardupilot's internal error models -->
-      <velocityOffset>0 0 0</velocityOffset>
-      <velocityDrift>0 0 0</velocityDrift>
-      <velocityDriftFrequency>0 0 0</velocityDriftFrequency>
-      <velocityGaussianNoise>0 0 0</velocityGaussianNoise>
-      <velocityScaleError>1 1 1</velocityScaleError>
-      <!-- Note:
-        The velocity Z does not really make sense, it is not used by
-        Ardupilot (right?).
-        However Z velocity drift is added to the Z position drift. -->
-      <!-- Explanations:
-         offset:          constant added to the real value
-         gaussian noise:  randomly generated noise added to the real value
-         drift:           amount of drift
-         drift frequency: time constant (as a frequency) for the drift
-         scale error:     scaling of the real value (before adding other noises)
-       -->
-    </plugin>
-  </gazebo>
+	<arg name="nspace" default=""/>
+	<arg name="bot" default=""/>
+	<xacro:include filename="$(find rotors_description)/urdf/component_snippets.xacro" />
+	<!-- Instantiate erlecopter "mechanics" -->
+	<xacro:include filename="$(find ardupilot_sitl_gazebo_plugin)/urdf/erlecopter.xacro" />
+	<!-- Specify reference parameters for GNSS receiver. -->
+	<xacro:include filename="$(find ardupilot_sitl_gazebo_plugin)/urdf/gps_home_location.xacro" />
+	<!-- Reference heading is equivalent to rotating Gazebo's map.
+		We do not use it for we would loose the match X=North, Y=West -->
+	<!-- in degrees, 0 so North is towards positive X values, and East is towards negative Y values -->
+	<xacro:property name="referenceHeading" value="0" />
+	<!-- Instantiate a controller. -->
+	<xacro:controller_plugin_macro namespace="${namespace}" imu_sub_topic="$(arg nspace)/imu"/>
+	<!-- Mount an ADIS16448 IMU. -->
+	<xacro:imu_plugin_macro
+		namespace="${namespace}"
+		imu_suffix=""
+		parent_link="base_link"
+		imu_topic="imu"
+		mass_imu_sensor="0.015"
+		gyroscope_noise_density="0.0003394"
+		gyroscopoe_random_walk="0.000038785"
+		gyroscope_bias_correlation_time="1000.0"
+		gyroscope_turn_on_bias_sigma="0.0087"
+		accelerometer_noise_density="0.004"
+		accelerometer_random_walk="0.006"
+		accelerometer_bias_correlation_time="300.0"
+		accelerometer_turn_on_bias_sigma="0.1960"
+	>
+		<inertia ixx="0.00001" ixy="0.0" ixz="0.0" iyy="0.00001" iyz="0.0" izz="0.00001" />
+		<origin xyz="0 0 0" rpy="0 0 0" />
+	</xacro:imu_plugin_macro>
+	<!-- Mount a GNSS receiver. -->
+	<gazebo>
+		<plugin name="${bot_name}_gps_sim" filename="libhector_gazebo_ros_gps.so">
+			<alwaysOn>true</alwaysOn>
+			<topicName>${bot_name}/fix</topicName>
+			<velocityTopicName>${bot_name}/fix_velocity</velocityTopicName>
+			<referenceLatitude>${referenceLatitude}</referenceLatitude>
+			<referenceLongitude>${referenceLongitude}</referenceLongitude>
+			<referenceHeading>${referenceHeading}</referenceHeading>
+			<referenceAltitude>${referenceAltitude}</referenceAltitude>
+			<!-- Sensor errors model for GPS Position measures -->
+			<!-- Units: [m], and [1/s] for drift frequency -->
+			<!-- For now, use Ardupilot's internal error models -->
+			<offset>0 0 0</offset>
+			<drift>0 0 0</drift>
+			<driftFrequency>0 0 0</driftFrequency>
+			<gaussianNoise>0 0 0</gaussianNoise>
+			<scaleError>1 1 1</scaleError>
+			<!-- Note:
+				For the moment there is no barometer, so axis Z of the GPS is
+				used as a barometer sensor (with the according error model) -->
+			<!-- Sensor errors model for GPS Velocity measures -->
+			<!-- Units: [m/s], and [1/s] for drift frequency -->
+			<!-- For now, use Ardupilot's internal error models -->
+			<velocityOffset>0 0 0</velocityOffset>
+			<velocityDrift>0 0 0</velocityDrift>
+			<velocityDriftFrequency>0 0 0</velocityDriftFrequency>
+			<velocityGaussianNoise>0 0 0</velocityGaussianNoise>
+			<velocityScaleError>1 1 1</velocityScaleError>
+			<!-- Note:
+				The velocity Z does not really make sense, it is not used by
+				Ardupilot (right?).
+				However Z velocity drift is added to the Z position drift. -->
+			<!-- Explanations:
+				offset:          constant added to the real value
+				gaussian noise:  randomly generated noise added to the real value
+				drift:           amount of drift
+				drift frequency: time constant (as a frequency) for the drift
+				scale error:     scaling of the real value (before adding other noises)
+			-->
+		</plugin>
+	</gazebo>
   <xacro:if value="$(arg enable_ground_truth)">
     <!-- Mount an IMU providing ground truth. -->
     <xacro:imu_plugin_macro
       namespace="${namespace}"
-      imu_suffix="gt"
+      imu_suffix="_gt"
       parent_link="base_link"
       imu_topic="ground_truth/imu"
@@ -100,5 +98,5 @@
     <xacro:odometry_plugin_macro
       namespace="${namespace}/ground_truth"
-      odometry_sensor_suffix="gt"
+      odometry_sensor_suffix="_gt"
       parent_link="base_link"
       pose_topic="pose"

File: ardupilot_sitl_gazebo_plugin/urdf/sensors/lidar_sensor.urdf.xacro (robot description, xacro)
@@ -18,5 +18,5 @@
           <!--<box size="0.01 0.01 0.01" /> -->
           <!-- <mesh filename="package://rotors_description/meshes/sonar_sensor/max_sonar_ez4.dae"/> -->
-           <!--<mesh filename="package://ardupilot_sitl_gazebo_plugin/meshes/${sensor_mesh}"/>-->
+           <mesh filename="package://ardupilot_sitl_gazebo_plugin/meshes/${sensor_mesh}"/>
          <!-- <mesh filename="package://ardupilot_sitl_gazebo_plugin/meshes/lidar_lite_v2/meshes/lidar_lite_v2.dae"/> -->
         </geometry>
